Commit message: fix

File: resources/robots/bdx/go_bdx.urdf (robot description, URDF)
Before this commit: robot bdx, 24 links, 23 joints
Links:
- removed link ear_left
- removed link ear_right
- removed link head
- removed link head_body_pitch
- removed link head_body_roll
- removed link head_body_yaw
- removed link neck
Joints:
- removed joint head_frame
- removed joint head_pitch
- removed joint head_roll
- removed joint head_yaw
- removed joint left_antenna
- removed joint neck_pitch
- removed joint right_antenna

Commit message: fix

File: resources/robots/bdx/go_bdx.urdf (robot description, URDF)
Before this commit: robot bdx, 17 links, 16 joints
Links:
- link pelvis: geometry visual mesh filename=meshes/pelvis.stl scale=0.001 0.001 0.001
